Commit message: Add USD configuration files for Hunter robot
- Created hunter_physics.usd to define the physical properties and structure of the Hunter robot.
- Created hunter_sensor.usd to specify the sensor configurations and parameters for the Hunter robot.

File: humanoidverse/data/robots/pdd/pdd.urdf (robot description, URDF)
Before this commit: robot pdd, 12 links, 11 joints
Links:
- link base_link: geometry collision box size=0.184 0.15 0.2; visual mesh filename=meshes/base_link.STL
- link leg_l1_link: geometry visual mesh filename=meshes/leg_l1_link.STL
- link leg_l2_link: geometry collision cylinder length=0.146 radius=0.065; visual mesh filename=meshes/leg_l2_link.STL
- link leg_l3_link: geometry collision box size=0.06 0.25 0.05; visual mesh filename=meshes/leg_l3_link.STL
- link leg_l4_link: geometry collision box size=0.041 0.25 0.03; collision cylinder length=0.07 radius=0.034
- link leg_l5_link: geometry collision box size=0.1001 0.0345 0.0175; visual mesh filename=meshes/leg_l5_link.STL
- link leg_r1_link: geometry visual mesh filename=meshes/leg_r1_link.STL
- link leg_r2_link: geometry collision cylinder length=0.146 radius=0.065; visual mesh filename=meshes/leg_r2_link.STL
- link leg_r3_link: geometry collision box size=0.06 0.25 0.05; visual mesh filename=meshes/leg_r3_link.STL
- link leg_r4_link: geometry collision box size=0.041 0.25 0.03; collision cylinder length=0.07 radius=0.034
- link leg_r5_link: geometry collision box size=0.1001 0.0345 0.0175; visual mesh filename=meshes/leg_r5_link.STL
