Commit message: Rename IMU joint and link for consistency in hunter URDF file

File: humanoidverse/data/robots/hunter/hunter.urdf (robot description, URDF)
Before this commit: robot hunter, 12 links, 11 joints
Links:
- removed link base_imu
- added link imu_link, mass 0.01; visual box size=0.015 0.015 0.004
Joints:
- removed joint base_imu_joint
- added joint imu_joint: type fixed, parent pelvis, child imu_link, origin xyz=0. 0. 0 rpy=0. 0. 0.

Commit message: Update evaluation command and configuration for Hunter: adjust model checkpoint paths, lower joint limits, and regenerate asset files

File: humanoidverse/data/robots/hunter/hunter.urdf (robot description, URDF)
Before this commit: robot hunter, 12 links, 11 joints
Joints:
- joint right_hip_yaw_joint: axis 0 0 1 -> 0 0 -1; limit lower=-1 upper=0.5 effort=23.7 velocity=30.1 -> lower=-0.5 upper=1 effort=23.7 velocity=30.1
